File: hardware/tinypad.kicad_pcb (KiCad board)
At the start: 2 copper layers, 60 x 28 mm, 25 parts, among them IC1 CD74HC147PWR, J1 Conn_01x06_Female, J2 CSP-USC16-TR, SW1 SW_Push, SW2 SW_Push, SW3 SW_Push, U1 ATtiny85-20SU

Commit message: Fixing minor wiring issues
Parts:
- turned C3 to 0 degrees
- turned D3 to 180 degrees
Routing:
- net VCC: track 182.4 -> 180.2 mm
- net GND: track 193.9 -> 194.9 mm
Changed lines of the file:
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@@
     (thickness 1.6)
     (drawings 36)
-    (tracks 346)
+    (tracks 351)
     (zones 0)
     (modules 25)
@@
   )
   (module LED_SMD:LED_SK6812MINI_PLCC4_3.5x3.5mm_P1.75mm (layer B.Cu)
-    (at 11.8508 18.4756)
+    (at 11.8508 18.4756 180)
     (descr https://cdn-shop.adafruit.com/product-files/2686/SK6812MINI_REV.01-1-2.pdf)
     (tags "LED RGB NeoPixel Mini")
@@
       (effects (font (size 1 1) (thickness 0.15)) (justify mirror))
     )
-    (pad 3 smd rect (at -1.75 0.875) (size 2 0.85) (layers B.Cu B.Paste B.Mask)
+    (pad 3 smd rect (at -1.75 0.875 180) (size 2 0.85) (layers B.Cu B.Paste B.Mask)
       (net 5 "Net-(D2-Pad1)"))
-    (pad 2 smd rect (at -1.75 -0.875) (size 2 0.85) (layers B.Cu B.Paste B.Mask)
+    (pad 2 smd rect (at -1.75 -0.875 180) (size 2 0.85) (layers B.Cu B.Paste B.Mask)
       (net 1 GND))
-    (pad 4 smd rect (at 1.75 0.875) (size 2 0.85) (layers B.Cu B.Paste B.Mask)
-      (net 2 VCC))
-    (pad 1 smd rect (at 1.75 -0.875) (size 2 0.85) (layers B.Cu B.Paste B.Mask)
+    (pad 4 smd rect (at 1.75 0.875 180) (size 2 0.85) (layers B.Cu B.Paste B.Mask)
+      (net 2 VCC))
+    (pad 1 smd rect (at 1.75 -0.875 180) (size 2 0.85) (layers B.Cu B.Paste B.Mask)
       (net 6 "Net-(D3-Pad1)"))
     (model ${KISYS3DMOD}/LED_SMD.3dshapes/LED_SK6812MINI_PLCC4_3.5x3.5mm_P1.75mm.wrl
@@
       (at (xyz 0 0 0))
       (scale (xyz 1 1 1))
-      (rotate (xyz 0 0 0))
+      (rotate (xyz 0 0 180))
     )
   )
@@
       (at (xyz 0 0 0))
       (scale (xyz 1 1 1))
-      (rotate (xyz 0 0 0))
+      (rotate (xyz 0 0 180))
     )
   )
@@
   )
   (module Capacitor_SMD:C_0805_2012Metric_Pad1.18x1.45mm_HandSolder (layer B.Cu)
-    (at 11.6508 22.2756 180)
+    (at 11.6508 22.2756)
     (descr "Capacitor SMD 0805 (2012 Metric), square (rectangular) end terminal, IPC_7351 nominal with elongated pad for handsoldering. (Body size source: IPC-SM-782 page 76, https://www.pcb-3d.com/wordpress/wp-content/uploads/ipc-sm-782a_amendment_1_and_2.pdf, https://docs.google.com/spreadsheets/d/1BsfQQcO9C6DZCsRaXUlFlo91Tg2WpOkGARC1WS5S8t0/edit?usp=sharing), generated with kicad-footprint-generator")
     (tags "capacitor handsolder")
@@
       (effects (font (size 0.5 0.5) (thickness 0.08)) (justify mirror))
     )
-    (pad 2 smd roundrect (at 1.0375 0 180) (size 1.175 1.45) (layers B.Cu B.Paste B.Mask) (roundrect_rratio 0.2127659574468085)
+    (pad 2 smd roundrect (at 1.0375 0) (size 1.175 1.45) (layers B.Cu B.Paste B.Mask) (roundrect_rratio 0.2127659574468085)
       (net 1 GND))
-    (pad 1 smd roundrect (at -1.0375 0 180) (size 1.175 1.45) (layers B.Cu B.Paste B.Mask) (roundrect_rratio 0.2127659574468085)
+    (pad 1 smd roundrect (at -1.0375 0) (size 1.175 1.45) (layers B.Cu B.Paste B.Mask) (roundrect_rratio 0.2127659574468085)
       (net 2 VCC))
     (model ${KISYS3DMOD}/Capacitor_SMD.3dshapes/C_0805_2012Metric.wrl
@@
   (via (at 45.4508 20.8756) (size 0.8) (drill 0.4) (layers F.Cu B.Cu) (net 1))
   (segment (start 27.5258 17.4006) (end 27.5258 17.4006) (width 0.25) (layer B.Cu) (net 1))
-  (via (at 27.5258 17.4006) (size 0.8) (drill 0.4) (layers F.Cu B.Cu) (net 1) (status 1000000))
+  (via (at 27.5258 17.4006) (size 0.8) (drill 0.4) (layers F.Cu B.Cu) (net 1))
   (segment (start 32.2883 21.8756) (end 32.8758 21.8756) (width 0.25) (layer B.Cu) (net 1))
   (segment (start 33.82581 19.77561) (end 33.2008 19.1506) (width 0.25) (layer B.Cu) (net 1))
@@
   (segment (start 27.5258 19.080944) (end 32.502845 24.057989) (width 0.25) (layer F.Cu) (net 1))
   (segment (start 27.5258 17.4006) (end 27.5258 19.080944) (width 0.25) (layer F.Cu) (net 1))
-  (segment (start 10.1008 17.6006) (end 8.7258 17.6006) (width 0.25) (layer B.Cu) (net 1))
+  (segment (start 10.1008 17.6006) (end 8.7258 17.6006) (width 0.25) (layer B.Cu) (net 2))
   (segment (start 55.1258 19.3506) (end 55.1258 20.22451) (width 0.25) (layer B.Cu) (net 1))
   (segment (start 53.62581 19.3506) (end 55.1258 19.3506) (width 0.25) (layer B.Cu) (net 1))
@@
   (segment (start 45.4508 20.3758) (end 33.995 8.92) (width 0.25) (layer F.Cu) (net 1))
   (segment (start 45.4508 20.8756) (end 45.4508 20.3758) (width 0.25) (layer F.Cu) (net 1))
-  (segment (start 10.6133 22.2756) (end 7.3377 19) (width 0.25) (layer B.Cu) (net 1))
   (segment (start 21.175011 19.324989) (end 20.65 19.85) (width 0.25) (layer B.Cu) (net 2))
   (segment (start 25.15 20.67) (end 25.45 20.67) (width 0.25) (layer B.Cu) (net 2))
@@
   (segment (start 22.613792 7.07541) (end 23.706202 5.983) (width 0.25) (layer B.Cu) (net 2))
   (segment (start 50.728361 10.495001) (end 54.403503 10.495001) (width 0.25) (layer F.Cu) (net 2))
-  (segment (start 15.4506 19.3506) (end 15.4506 19.5133) (width 0.25) (layer B.Cu) (net 2))
   (segment (start 18.0016 6.0504) (end 19.02661 7.07541) (width 0.25) (layer B.Cu) (net 2))
   (segment (start 23.706202 5.983) (end 29.84 5.983) (width 0.25) (layer B.Cu) (net 2))
@@
   (via (at 46.2688 6.03544) (size 0.8) (drill 0.4) (layers F.Cu B.Cu) (net 2))
   (segment (start 55.575801 18.582599) (end 55.575801 19.138099) (width 0.25) (layer B.Cu) (net 2))
-  (segment (start 13.6008 19.3506) (end 15.4506 19.3506) (width 0.25) (layer B.Cu) (net 2))
   (segment (start 39.8025 1.763) (end 39.727499 1.838001) (width 0.25) (layer B.Cu) (net 2))
   (segment (start 40.79 1.763) (end 39.8025 1.763) (width 0.25) (layer B.Cu) (net 2))
@@
   (segment (start 47.9758 15.7258) (end 47.75 15.5) (width 0.25) (layer B.Cu) (net 2))
   (segment (start 47.9758 17.6006) (end 47.9758 15.7258) (width 0.25) (layer B.Cu) (net 2))
-  (segment (start 15.458001 23.708001) (end 14.120701 23.708001) (width 0.25) (layer B.Cu) (net 2))
-  (segment (start 10.03762 23.32561) (end 4.5 17.78799) (width 0.25) (layer B.Cu) (net 2))
-  (segment (start 12.36329 23.32561) (end 10.03762 23.32561) (width 0.25) (layer B.Cu) (net 2))
-  (segment (start 15.4506 19.3506) (end 15.4506 23.7006) (width 0.25) (layer B.Cu) (net 2))
-  (segment (start 12.6883 22.2756) (end 12.6883 23.0006) (width 0.25) (layer B.Cu) (net 2))
-  (segment (start 13.33831 22.92561) (end 12.6883 22.2756) (width 0.25) (layer B.Cu) (net 2))
-  (segment (start 12.6883 23.0006) (end 12.36329 23.32561) (width 0.25) (layer B.Cu) (net 2))
-  (segment (start 14.120701 23.708001) (end 12.6883 22.2756) (width 0.25) (layer B.Cu) (net 2))
+  (segment (start 12.6883 22.2756) (end 12.6883 23.0006) (width 0.25) (layer B.Cu) (net 1))
+  (segment (start 13.2758 22.2756) (end 15.25 20.3014) (width 0.25) (layer B.Cu) (net 1))
+  (segment (start 12.6883 22.2756) (end 13.2758 22.2756) (width 0.25) (layer B.Cu) (net 1))
+  (segment (start 15.25 20.3014) (end 15.25 19.5) (width 0.25) (layer B.Cu) (net 1))
+  (segment (start 13.6008 19.3506) (end 15.1006 19.3506) (width 0.25) (layer B.Cu) (net 1))
+  (segment (start 15.1006 19.3506) (end 15.5 19.75) (width 0.25) (layer B.Cu) (net 1))
+  (segment (start 10.420011 23.708001) (end 9.731005 23.018995) (width 0.25) (layer B.Cu) (net 2))
+  (segment (start 15.458001 23.708001) (end 10.420011 23.708001) (width 0.25) (layer B.Cu) (net 2))
+  (segment (start 10.03762 23.32561) (end 9.731005 23.018995) (width 0.25) (layer B.Cu) (net 2))
+  (segment (start 9.9744 22.2756) (end 9.481005 22.768995) (width 0.25) (layer B.Cu) (net 2))
+  (segment (start 10.6133 22.2756) (end 9.9744 22.2756) (width 0.25) (layer B.Cu) (net 2))
+  (segment (start 9.731005 23.018995) (end 9.481005 22.768995) (width 0.25) (layer B.Cu) (net 2))
+  (segment (start 8.7258 17.6006) (end 8.7258 18.0242) (width 0.25) (layer B.Cu) (net 2))
+  (segment (start 6.731005 20.018995) (end 4.5 17.78799) (width 0.25) (layer B.Cu) (net 2))
+  (segment (start 8.7258 18.0242) (end 6.731005 20.018995) (width 0.25) (layer B.Cu) (net 2))
+  (segment (start 9.481005 22.768995) (end 6.731005 20.018995) (width 0.25) (layer B.Cu) (net 2))
   (segment (start 33.2008 17.4006) (end 44.3758 17.4006) (width 0.25) (layer B.Cu) (net 3))
   (segment (start 44.3758 17.4006) (end 46.3258 19.3506) (width 0.25) (layer B.Cu) (net 3))
